File: hardware/pcb/imu.kicad_sch (KiCad schematic)
At the start: 3 parts, among them U2 LSM6DSV16XTR

Commit message: Changed GNDPWR to GND and changed GND to speciality GNDs
Connections:
- net INT1 renamed INT1_IMU
- net INT2 renamed INT2_IMU
Changed lines of the file:
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@@
 		)
 	)
-	(hierarchical_label "INT1"
+	(hierarchical_label "INT1_IMU"
 		(shape input)
 		(at 160.02 81.28 0)
@@
 		)
 	)
-	(hierarchical_label "INT2"
+	(hierarchical_label "INT2_IMU"
 		(shape input)
 		(at 160.02 83.82 0)
