File: hardware/pcb/gnss.kicad_sch (KiCad schematic)
At the start: 1 part, among them U4 MIA-M10Q-00B

Commit message: Update(hardware): Completed some schematics
Connections:
- net GNDPWR: now reaches U4.A1 (GND)
- net GNDPWR: now also U4.A2 (GND__1), U4.A3 (GND__2), U4.A8 (GND__3), U4.A9 (GND__4), U4.B2 (GND__5), U4.B8 (GND__6), U4.C3 (GND__7), U4.C9 (GND__8), U4.E3 (GND__9), U4.E4 (GND__10), U4.E9 (GND__11), U4.F1 (GND__12), U4.F3 (GND__13), U4.F4 (GND__14), U4.G3 (GND__15), U4.G4 (GND__16), U4.G5 (GND__17), U4.G6 (GND__18), U4.H8 (GND__19), U4.J8 (GND__20), U4.J9 (GND__21)

Commit message: Changed GNDPWR to GND and changed GND to speciality GNDs
Connections:
- net GNDPWR renamed GND
Changed lines of the file:
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@@
 	)
 	(symbol
-		(lib_id "power:GNDPWR")
+		(lib_id "power:GND")
 		(at 127 165.1 0)
 		(unit 1)
@@
 		(fields_autoplaced yes)
 		(property "Reference" "#PWR027"
-			(at 127 170.18 0)
+			(at 127 171.45 0)
 			(hide yes)
 			(show_name no)
@@
 			)
 		)
-		(property "Value" "GNDPWR"
-			(at 126.873 168.91 0)
+		(property "Value" "GND"
+			(at 127 170.18 0)
 			(show_name no)
 			(do_not_autoplace no)
@@
 		)
 		(property "Footprint" ""
-			(at 127 166.37 0)
+			(at 127 165.1 0)
 			(hide yes)
 			(show_name no)
@@
 		)
 		(property "Datasheet" ""
-			(at 127 166.37 0)
+			(at 127 165.1 0)
 			(hide yes)
 			(show_name no)
@@
 			)
 		)
-		(property "Description" "Power symbol creates a global label with name \"GNDPWR\" , global ground"
+		(property "Description" "Power symbol creates a global label with name \"GND\" , ground"
 			(at 127 165.1 0)
 			(hide yes)

Commit message: Progress on 3V3 circuit versions.
Parts:
- removed U4: MIA-M10Q-00B, footprints:BGA53C50P9X9_450X450X100, symbol symbols:MIA-M10Q-00B
- added E1: SR4G008, footprints:XCVR_SR4G008, symbol symbols:SR4G008
- added TP1: TestPoint_Square, symbol Connector:TestPoint_Square
- added U4: TCK127BG_LF, footprints:WCSP4G_TOS, symbol symbols:TCK127BG_LF
- added U9: MAX-M10M-00B, footprints:XCVR_MAX-M10M-00B, symbol symbols:MAX-M10M-00B
Connections:
- net GND: now also E1.3, E1.4, E1.6, U4.B1 (GND), U9.1 (GND), U9.10 (GND__1), U9.12 (GND__2)
- new net: E1.2, U9.11 (RF_IN)
- new net: TP1.1, U9.18 (~{SAFEBOOT})
- new net: U4.A1 (VOUT), U9.7 (V_IO), U9.8 (VCC)
- new net +3V3: U4.A2 (VIN)
- new net GNSS_EN: U4.B2 (CONTROL)
- new net GNSS_EXTINT: U9.5 (EXTINT)
- new net GNSS_RESET: U9.9 (~{RESET})
- new net GNSS_RXD: U9.3 (RXD)
- new net GNSS_TIMEPULSE: U9.4 (TIMEPULSE)
- new net GNSS_TXD: U9.2 (TXD)
- no-connect marks 0 -> 6
