File: hardware/pcb/speaker.kicad_sch (KiCad schematic)
At the start: 0 parts

Commit message: Progress on 3V3 circuit versions.
Parts:
- added LS1: CMS-151125-18S-X8, footprints:SPKR_CMS-151125-18S-X8, symbol symbols:CMS-151125-18S-X8
- added U11: PAM8013AKR, footprints.PAM8013AKR, symbol symbols:PAM8013AKR
Connections:
- new net +3V3: U11.4 (VDD), U11.5 (VDD)
- new net GND: U11.2 (GND), U11.6 (GND)
- new net SPEAKER_N: U11.7 (INN)
- new net SPEAKER_P: U11.1 (INP)
