File: hardware/pcb/barometer.kicad_sch (KiCad schematic)
At the start: 1 part, among them U6 BMP581

Commit message: Update(hardware): Completed some schematics
Parts:
- added C3, C4: 100n, Package_SO:SOIC-8_3.9x4.9mm_P1.27mm, symbol Device:C
Connections:
- net INT: now also U6.7 (INT)
- net SCK: now also U6.2 (SCK)
- net SDA: now also U6.4 (SDI)
- net +1V8: now reaches U6.1 (VDDIO)
- net +1V8: now also U6.10 (VDD), U6.5 (SDO), U6.6 (CSB), C3.1, C4.1
- net GNDPWR: now reaches U6.3 (VSS_1)
- net GNDPWR: now also U6.8 (VSS_2), U6.9 (VSS_3), C3.2, C4.2
Other:
- note added: "Documentation available from here"
- note added: "Example Sparkfun board"
- moved on the sheet: U6

Commit message: Changed GNDPWR to GND and changed GND to speciality GNDs
Connections:
- net GNDPWR renamed GND
- net INT renamed INT_BARO

Commit message: Update(hardware): Schematic changes
Connections:
- net +1V8 renamed +3V3
- net +3V3: no longer U6.6 (CSB)
- no-connect marks 0 -> 1
